Commit message: Update robot configuration and launch files for improved simulation accuracy
- Adjust wheel separation and radius in controllers.yaml for better movement dynamics.
- Modify URDF properties for wheel dimensions and track widths to match new configuration and tune friction for skid-steering.
- Update launch file to include additional Gazebo initialization parameters and adjust spawn height.

File: src/beach_robot_description/urdf/beach_robot.urdf.xacro (robot description, xacro)
@@ -4,10 +4,11 @@
        Defaults (tune later)
        ========================= -->
-  <xacro:property name="wheel_radius" value="0.15"/>
+  <xacro:property name="wheel_radius" value="0.165"/>
   <xacro:property name="wheel_width"  value="0.08"/>
-  <xacro:property name="wheelbase"    value="0.80"/>
-  <xacro:property name="track_width"  value="0.60"/>
-  <xacro:property name="base_length"  value="1.00"/>
-  <xacro:property name="base_width"   value="0.70"/>
+  <xacro:property name="wheelbase"    value="0.975"/>
+  <xacro:property name="front_track_width" value="0.75"/>
+  <xacro:property name="rear_track_width"  value="1.17"/>
+  <xacro:property name="base_length"  value="1.20"/>
+  <xacro:property name="base_width"   value="1.30"/>
   <xacro:property name="base_height"  value="0.25"/>
   <!-- frames -->
@@ -55,5 +56,5 @@
        Wheel macro
        ========================= -->
-  <xacro:macro name="wheel" params="name x y">
+  <xacro:macro name="wheel" params="name x y axis_sign:=1">
     <link name="${name}_link">
       <inertial>
@@ -80,12 +81,46 @@
         <!-- wheel center at chassis bottom plane -->
         <origin xyz="${x} ${y} ${-base_height/2}" rpy="0 0 0"/>
-        <axis xyz="0 1 0"/>
+        <axis xyz="0 ${axis_sign} 0"/>
+        <limit effort="20.0" velocity="50.0"/>
       </joint>
   </xacro:macro>
   <!-- 4 wheels (front pair = tracks in real life, but in sim treat as wheels for skid-drive) -->
-  <xacro:wheel name="front_left"  x="${ wheelbase/2}" y="${ track_width/2}"/>
-  <xacro:wheel name="front_right" x="${ wheelbase/2}" y="${-track_width/2}"/>
-  <xacro:wheel name="rear_left"   x="${-wheelbase/2}" y="${ track_width/2}"/>
-  <xacro:wheel name="rear_right"  x="${-wheelbase/2}" y="${-track_width/2}"/>
+  <xacro:wheel name="front_left"  x="${ wheelbase/2}" y="${ front_track_width/2}" axis_sign="1"/>
+  <xacro:wheel name="front_right" x="${ wheelbase/2}" y="${-front_track_width/2}" axis_sign="1"/>
+  <xacro:wheel name="rear_left"   x="${-wheelbase/2}" y="${ rear_track_width/2}" axis_sign="1"/>
+  <xacro:wheel name="rear_right"  x="${-wheelbase/2}" y="${-rear_track_width/2}" axis_sign="1"/>
+  <!-- <xacro:wheel name="rear_left"   x="${-wheelbase/2}" y="${ front_track_width/2}" axis_sign="1"/>
+  <xacro:wheel name="rear_right"  x="${-wheelbase/2}" y="${-front_track_width/2}" axis_sign="1"/> -->
+  <!-- <xacro:macro name="wheel_friction" params="link_name">
+    <gazebo reference="${link_name}">
+      <mu1>1.0</mu1>
+      <mu2>1.0</mu2>
+      <kp>1000000.0</kp>
+      <kd>10.0</kd>
+    </gazebo>
+  </xacro:macro>
+  <xacro:wheel_friction link_name="front_left_link"/>
+  <xacro:wheel_friction link_name="rear_left_link"/>
+  <xacro:wheel_friction link_name="front_right_link"/>
+  <xacro:wheel_friction link_name="rear_right_link"/> -->
+  <xacro:macro name="wheel_contact" params="link
+                                           mu_roll:=0.8 mu_lat:=0.12
+                                           slip_roll:=0.0 slip_lat:=0.25
+                                           kp:=5000000 kd:=80.0">
+    <gazebo reference="${link}">
+      <!-- ลด mu2 / เพิ่ม slip2 เพื่อมให้เลี้ยวง่ายขึ้น -->
+      <mu1>${mu_roll}</mu1>
+      <mu2>${mu_lat}</mu2>
+      <kp>${kp}</kp>
+      <kd>${kd}</kd>
+      <fdir1>1 0 0</fdir1>
+      <slip1>${slip_roll}</slip1>
+      <slip2>${slip_lat}</slip2>
+    </gazebo>
+  </xacro:macro>
+  <xacro:wheel_contact link="front_left_link"/>
+  <xacro:wheel_contact link="front_right_link"/>
+  <xacro:wheel_contact link="rear_left_link"/>
+  <xacro:wheel_contact link="rear_right_link"/>
   <!-- =========================
        Sensor frames (static)
@@ -216,5 +251,5 @@
     </sensor>
   </gazebo>
-  <gazebo reference="front_left_link">
+  <!-- <gazebo reference="front_left_link">
     <mu1>1.0</mu1>
     <mu2>1.0</mu2>
@@ -231,5 +266,5 @@
     <mu1>1.0</mu1>
     <mu2>1.0</mu2>
-  </gazebo>
+  </gazebo> -->
   <!-- Ultrasonic sensors (range) -->
   <xacro:macro name="ultrasonic" params="ref name topic">
